File: electronics/ofen.kicad_sch (KiCad schematic)
At the start: 55 parts, among them IC1 TS4061BILT-1.225, IC2 MCP3461T-E_ST, J1 Conn_02x03_Odd_Even, J2 Conn_01x04, J3 Conn_01x05, J4 Conn_01x04, J5 Conn_01x02, J6 DB9_Female_MountingHoles, K1 RAYEX-L90AS, Q1 BC337, SW1 SW_Coded, U1 LD1086DT33TR, U2 ILI9488, U3 CD4097B, U4 ATmega328P-A, U5 Keypad_4x4, U6 74HC165, U7 4017

Commit message: updated to version 2.1 of the pcb and added the first steps of the firmware
Parts:
- removed C17: 22n, Capacitor_THT:C_Disc_D5.0mm_W2.5mm_P2.50mm, symbol Device:C
- removed D5, D6: D, Diode_THT:D_A-405_P7.62mm_Horizontal, symbol Device:D
- removed J2, J4: Conn_01x04, Connector_PinHeader_2.54mm:PinHeader_1x04_P2.54mm_Vertical, symbol Connector_Generic:Conn_01x04
- removed JP1: SolderJumper_2_Open, Jumper:SolderJumper-2_P1.3mm_Open_RoundedPad1.0x1.5mm, symbol Jumper:SolderJumper_2_Open
- removed JP5: SolderJumper_3_Open, Jumper:SolderJumper-3_P1.3mm_Open_RoundedPad1.0x1.5mm_NumberLabels, symbol Jumper:SolderJumper_3_Open
- removed R14: 15k, Resistor_THT:R_Axial_DIN0207_L6.3mm_D2.5mm_P10.16mm_Horizontal, symbol ofen:R
- removed U2: ILI9488, ofen_v2:ribbon_1x17_vertical, symbol ofen:ILI9488
- removed U7: 4017, Package_DIP:DIP-16_W7.62mm, symbol 4xxx:4017
- added C10: 10µ, Capacitor_THT:CP_Radial_Tantal_D4.5mm_P5.00mm, symbol Device:C_Polarized
- added C3, C4, C6: 22n, Capacitor_THT:C_Disc_D5.0mm_W2.5mm_P2.50mm, symbol Device:C
- added J1: LEDs, Connector_Molex:Molex_KK-254_AE-6410-04A_1x04_P2.54mm_Vertical, symbol Connector_Generic:Conn_01x04
- added J4: CH0, Connector_PinHeader_2.54mm:PinHeader_1x03_P2.54mm_Vertical, symbol Connector_Generic:Conn_01x03
- added J5: CH1, Connector_PinHeader_2.54mm:PinHeader_1x03_P2.54mm_Vertical, symbol Connector_Generic:Conn_01x03
- added J8: RST, Connector_PinHeader_2.54mm:PinHeader_1x01_P2.54mm_Vertical, symbol Connector_Generic:Conn_01x01
- added RN1, RN2: 223, Resistor_SMD:R_Array_Concave_4x0603, symbol Device:R_Pack04
- added SW2: RST, Button_Switch_THT:SW_Tactile_SPST_Angled_PTS645Vx83-2LFS, symbol Switch:SW_Push
- added U4: SD_card, Connector_Molex:Molex_Micro-Latch_53253-0470_1x04_P2.00mm_Vertical, symbol ofen:SD_card
- added U6: ILI9488, ofen_v2:ribbon_1x10_horizontal, symbol ofen:ILI9488
- added U7: 74HC238, Package_SO:SOP-16_3.9x9.9mm_P1.27mm, symbol 74xx:74HC238
- IC2: value MCP3461T-E_ST -> MCP3461
- J3: renamed from J5; value Conn_01x02 -> 12VDC
- J6: renamed from J3; value Conn_01x05 -> UART
- J7: renamed from J1; value Conn_02x03_Odd_Even -> ISP
- JP1: renamed from JP2; value SolderJumper_2_Open -> Y5
- JP2: renamed from JP3; value SolderJumper_2_Open -> Y6
- JP3: renamed from JP4; value SolderJumper_2_Open -> Y7
- K1: value RAYEX-L90AS -> HF2160-1A-12DE
- R13: value 180 -> 2,2k
- SW1: footprint Connector_PinHeader_2.54mm:PinHeader_1x04_P2.54mm_Vertical -> Connector_Molex:Molex_Micro-Latch_53253-0470_1x04_P2.00mm_Vertical
- U1: value LD1086DT33TR -> CYT8117T33
- U5: footprint Connector_Molex:Molex_Micro-Latch_53254-0870_1x08_P2.00mm_Horizontal -> Connector_Molex:Molex_Micro-Latch_53253-0870_1x08_P2.00mm_Vertical
- U8: renamed from U4; value ATmega328P-A -> ATmega328P
- renumbered C4 to C11, C7 to C12, C10 to C13, C11 to C14, C13 to C15, C15 to C16, C14 to C17, C16 to C18, C8 to C2, C12 to C5, C2 to C7, C9 to C8, C3 to C9, D2 to D1, J6 to J2, R12 to R1, R9 to R10, R4 to R11, R7 to R12, R1 to R2, R6 to R3, R10 to R4, R11 to R5, R2 to R6, R5 to R7, R3 to R9, U3 to U2, U6 to U3
Connections:
- net +3.3V: now also J7.2 (Pin_2), R13.1, RN1.6 (R3.2), RN1.7 (R2.2), RN1.8 (R1.2), U6.1 (3V3), U7.16 (VCC), U7.6 (E3); no longer J6.3 (Pin_3)
- net GND: now also C10.2, C4.2, C6.2, J1.1 (Pin_1), RN2.1 (R1.1), RN2.2 (R2.1), RN2.3 (R3.1), RN2.4 (R4.1), SW2.1, U6.2 (GND), U7.3 (A2), U7.4 (~{E1}), U7.5 (~{E2}), U7.8 (GND)
- net at U2.10 (A): now also U8.27 (PC4); no longer U8.8 (XTAL2/PB7)
- net at U2.11 (B): now also U8.26 (PC3); no longer U8.9 (PD5)
- net at U2.14 (C): now also U8.25 (PC2)
- net at JP3.1 (A), U2.15 (Y7): now also J5.3 (Pin_3)
- net at JP2.1 (A), U2.16 (Y6): now also J5.2 (Pin_2)
- net at JP1.1 (A), U2.18 (Y5): now also J5.1 (Pin_1)
- net at U2.19 (Y4): now also J2.7, R7.2
- net at U2.2 (X7): now also J4.3 (Pin_3)
- net at C2.1, J2.9, U2.21 (Y2): now also C3.2
- net at U2.3 (X6): now also J4.2 (Pin_2)
- net at U2.4 (X5): now also J4.1 (Pin_1)
- net at U2.5 (X4): now also J2.2
- net at C8.1, R7.1, R8.2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: now also C6.1
- net at C2.2, R3.1, U2.7 (X2): now also C3.1
- net at C5.1, R10.1, R9.2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: now also C4.1
- net at J2.3, R4.2, SW1.2 (D0)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: now also J1.2 (Pin_2), RN1.3 (R3.1)
- net at SW1.3 (D1), U3.12 (D1): now also RN1.2 (R2.1)
- net at SW1.4 (D2), U3.13 (D2): now also RN1.1 (R1.1)
- net at C15.1, U3.14 (D3), U5.5: now also RN2.8 (R1.2)
- net at U5.1: now also U7.15 (Y0)
- net at U5.2: now also U7.14 (Y1)
- net at U5.3: now also U7.13 (Y2)
- net at U5.4: now also U7.12 (Y3)
- net at C16.1, U3.3 (D4), U5.6: now also RN2.7 (R2.2)
- net at C17.1, U3.4 (D5), U5.7: now also RN2.6 (R3.2)
- net at C18.1, U3.5 (D6), U5.8: now also RN2.5 (R4.2)
- net at U3.1 (~{PL}): now also U8.7 (XTAL1/PB6); no longer R13.2
- net at U3.2 (CP): now also U8.8 (XTAL2/PB7); no longer U8.23 (PC0)
- net at U3.9 (Q7): now also U8.2 (PD4); no longer U8.22 (ADC7)
- net at C12.1, IC1.1 (K), J2.6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: now also C10.1
- net at IC2.14 (SCK), U8.17 (PB5): now also J7.3 (Pin_3), U4.4 (SCK), U6.7 (SCK)
- net at IC2.15 (SDI), J7.4 (Pin_4), U8.15 (PB3): now also U4.2 (SDI), U6.6 (SDI)
- net at IC2.16 (SDO), J7.1 (Pin_1), U8.16 (PB4): now also U4.3 (SDO), U6.8 (SDO)
- net at IC2.17 (~{IRQ}/MDAT): now also U8.1 (PD3); no longer U8.32 (PD2)
- net at U8.13 (PB1): now also U6.5 (D/C)
- net at U8.12 (PB0): now also U6.4 (RST)
- net at U8.11 (PD7): now also U6.3 (CS)
- net at U8.10 (PD6): now also U7.1 (A0)
- net at U8.28 (PC5): now also J2.4, R1.2, R5.1
- net at J7.5 (Pin_5), U8.29 (~{RESET}/PC6): now also R13.2, J8.1 (Pin_1), SW2.2
- net at U8.24 (PC1): now also IC2.13 (~{CS})
- net at R2.2: now also J1.3 (Pin_3); no longer J2.2
- net at R1.1: now also J1.4 (Pin_4); no longer J2.4
- new net: U7.2 (A1), U8.9 (PD5)
- new net: U4.1 (CS), U8.14 (PB2)
- new net: U6.9 (TCS), U8.23 (PC0)
- new net: U6.10 (TIRQ), U8.32 (PD2)
- no-connect marks 22 -> 16
Other:
- moved on the sheet: C1, C11, C15, C16, C17, C18, C2, C7, C8, C9, D1, J3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

Commit message: wip
Parts:
- removed C15, C16, C17, C18: 22n, Capacitor_THT:C_Disc_D5.0mm_W2.5mm_P2.50mm, symbol Device:C
